Commit message: messed it up now fixed

File: thorvald_nvidia/loki/loki_description/urdf/thorvald_model.xacro (robot description, xacro)
@@ -3,7 +3,7 @@
   <xacro:arg name="robot_name" default=""/>
   <xacro:arg name="tf_prefix" default=""/>
-  <xacro:arg name="robot_config" default="$(find-pkg-share loki_base)/config/robot_017.yaml"/>
+  <xacro:arg name="robot_config" default="$(find loki_base)/config/robot_017.yaml"/>
   <xacro:arg name="model_extras" default=""/>
-  <gazebo>
+  <!-- <gazebo>
     <plugin name="$(arg robot_name)_loki_gazebo_plugins" filename="libloki_gazebo_plugins_synch.so">
       <alwaysOn>true</alwaysOn>
@@ -37,5 +37,5 @@
       <wheel10>$(arg tf_prefix)wheel10</wheel10>
     </plugin>
-  </gazebo>
+  </gazebo> -->
    <xacro:macro name="cuboid_inertial" params="mass length width height xyz rpy">
     <inertial>
@@ -70,5 +70,5 @@
 <!-- ROBOT-SPECIFIC PARAMETERS -->
   <!-- Parameters file in config directory as specified in argument -->
-  <xacro:property name="base_params" value="${load_yaml('$(arg robot_config)')}"/>
+  <xacro:property name="base_params" value="${xacro.load_yaml('$(arg robot_config)')}"/>
   <xacro:property name="model_extras" value="$(arg model_extras)"/>
   <!-- MATERIAL DEFINITIONS -->
